File: Shield/Shield.sch (EAGLE design)
At the start: 25 parts

Commit message: Update Shield.sch
Parts:
- removed LED1, LED2, LED3, LED4, LED5, LED6, LED7, LED8: (no value), led:LED5MM
- removed PAD4: (no value), wirepad:2,15/1,0
- added U$1, U$2, U$3, U$4, U$5, U$6, U$7, U$8: LED5MM, fab:LED5MM
Connections:
- removed net N$16: PAD4.P, R6.2, R7.1, T1.S, T2.S, T3.S, T4.S, T5.S
- new net GND: PCB1.GND, PCB1.GND., PCB1.GND.., R6.2, R7.1, T1.S, T2.S, T3.S, T4.S, T5.S
- net N$1: now also U$1.C, U$2.A; no longer LED1.A, LED2.C
- net N$10: now also U$2.C; no longer LED1.C
- net N$11: now also U$5.C; no longer LED5.C
- net N$12: now also U$4.C; no longer LED4.C
- net N$14: now also U$7.C; no longer LED6.C
- net N$2: now also U$3.C, U$5.A; no longer LED3.C, LED5.A
- net N$3: now also U$4.A, U$8.C; no longer LED4.A, LED7.C
- net N$4: now also U$6.C, U$7.A; no longer LED6.A, LED8.C
- net N$5: now also U$1.A; no longer LED2.A
- net N$6: now also U$3.A; no longer LED3.A
- net N$7: now also U$8.A; no longer LED7.A
- net N$8: now also U$6.A; no longer LED8.A
Other:
- moved on the sheet: PAD1, PAD2, PAD3, R1, R2, R3, R4, R5, R6, R7, T1, T2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
